Commit message: added 500mm urdf and meshes

File: robot/ewellix_lift_std.urdf.xacro (robot description, xacro)
@@ -24,3 +24,8 @@
         </xacro:ewellix_lift_700mm>
     </xacro:if>
+    <xacro:if value="${lift_selector == 'lift_500mm'}">
+        <xacro:ewellix_lift_500mm prefix="$(arg prefix)" parent ="$(arg base_frame)" cut_model = "$(arg cut_model)" >
+            <origin xyz="0 0 0" rpy="0 0 0"/>
+        </xacro:ewellix_lift_500mm>
+    </xacro:if>
 </robot>
