Commit message: modified meshes and urdf of the 500mm model to have proper scale

File: urdf/ewellix_lift_500mm.urdf.xacro (robot description, xacro)
@@ -16,5 +16,5 @@
       </visual>
       <collision>
-        <origin xyz="-0.005 0 0.00235" rpy="0 0 0"/>
+        <origin xyz="0 0 0" rpy="0 0 0"/>
         <geometry>
           <mesh filename="package://ewellix_description/meshes/ewellix_lift_base_500mm.stl"/>
@@ -39,5 +39,5 @@
         <geometry>
           <xacro:if value="${cut_model}">
-            <mesh filename="package://ewellix_description/meshes/ewellix_lift_top_500mm_cut.stl"/>
+            <mesh filename="package://ewellix_description/meshes/ewellix_lift_top_500mm.stl"/>
           </xacro:if>
           <xacro:unless value="${cut_model}">
@@ -53,5 +53,5 @@
         <geometry>
           <xacro:if value="${cut_model}">
-            <mesh filename="package://ewellix_description/meshes/ewellix_lift_top_500mm_cut.stl"/>
+            <mesh filename="package://ewellix_description/meshes/ewellix_lift_top_500mm.stl"/>
           </xacro:if>
           <xacro:unless value="${cut_model}">
@@ -70,5 +70,5 @@
       <parent link="${prefix}ewellix_lift_base_link"/>
       <child link="${prefix}ewellix_lift_top_link" />
-      <origin xyz="0 0 0.54" rpy="0 0 0" />
+      <origin xyz="0 0 0.047" rpy="0 0 0" />
       <limit effort="1000" lower="0.0" upper="0.7" velocity="0.088"/>
       <axis xyz="0 0 1" />

Commit message: modified upper limit of the 500mm lifting unit

File: urdf/ewellix_lift_500mm.urdf.xacro (robot description, xacro)
@@ -71,5 +71,5 @@
       <child link="${prefix}ewellix_lift_top_link" />
       <origin xyz="0 0 0.047" rpy="0 0 0" />
-      <limit effort="1000" lower="0.0" upper="0.7" velocity="0.088"/>
+      <limit effort="1000" lower="0.0" upper="0.5" velocity="0.088"/>
       <axis xyz="0 0 1" />
     </joint>
